File: Eagle Files/Punktschweis_pulser.brd (EAGLE design)
At the start: 50 x 60 mm, 20 parts

Commit message: Added Gerber Files for pcbway.com
Routing:
- net N$3: track 123.5 -> 120.5 mm
Changed lines of the file:
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@@
 <wire x1="6.62" y1="52.28" x2="6.5" y2="52.28" width="0.6096" layer="1"/>
 <wire x1="6.5" y1="52.28" x2="6.5" y2="44.5" width="0.6096" layer="1"/>
-<wire x1="6.5" y1="44.5" x2="1" y2="44.5" width="0.6096" layer="1"/>
-<wire x1="1" y1="44.5" x2="1" y2="22.5" width="0.6096" layer="1"/>
-<wire x1="1" y1="22.5" x2="6.5" y2="22.5" width="0.6096" layer="1"/>
+<wire x1="6.5" y1="44.5" x2="2.5" y2="44.5" width="0.6096" layer="1"/>
+<wire x1="2.5" y1="44.5" x2="2.5" y2="22.5" width="0.6096" layer="1"/>
+<wire x1="2.5" y1="22.5" x2="6.5" y2="22.5" width="0.6096" layer="1"/>
 <wire x1="3.9015" y1="10.3275" x2="3.9015" y2="9.8685" width="0.254" layer="1"/>
 <wire x1="6.1965" y1="12.6225" x2="3.9015" y2="10.3275" width="0.254" layer="1"/>
@@
 <wire x1="16.983" y1="37.179" x2="16.78" y2="37.04" width="0.254" layer="1"/>
 <wire x1="5.2785" y1="11.016" x2="11.016" y2="5.2785" width="0.254" layer="16"/>
-<wire x1="3.672" y1="11.016" x2="5.2785" y2="11.016" width="0.254" layer="16"/>
-<wire x1="1.836" y1="12.852" x2="3.672" y2="11.016" width="0.254" layer="16"/>
-<wire x1="1.836" y1="37.8675" x2="1.836" y2="12.852" width="0.254" layer="16"/>
-<wire x1="3.213" y1="39.2445" x2="1.836" y2="37.8675" width="0.254" layer="16"/>
+<wire x1="2.672" y1="11.016" x2="5.2785" y2="11.016" width="0.254" layer="16"/>
+<wire x1="2.336" y1="12.852" x2="2.672" y2="11.016" width="0.254" layer="16"/>
+<wire x1="2.336" y1="37.8675" x2="2.336" y2="12.852" width="0.254" layer="16"/>
+<wire x1="3.213" y1="39.2445" x2="2.336" y2="37.8675" width="0.254" layer="16"/>
 <wire x1="14.688" y1="39.2445" x2="3.213" y2="39.2445" width="0.254" layer="16"/>
 <wire x1="16.7535" y1="37.179" x2="14.688" y2="39.2445" width="0.254" layer="16"/>
